File: proxy_ev.sch (KiCad schematic (older format))
At the start: 2 parts

Commit message: Add files via upload
Parts:
- added R303: 30k, Resistor_SMD:R_0603_1608Metric, symbol Device:R_Small_US
- added R304: 82k, Resistor_SMD:R_0603_1608Metric, symbol Device:R_Small_US
- R301: footprint (none) -> Resistor_SMD:R_0402_1005Metric
- R302: footprint (none) -> Resistor_SMD:R_0603_1608Metric
Connections:
- net GND: now also R304.2
- net PROXY: now also R303.1
- new net PROXY_SENS: R303.2, R304.1
Changed lines of the file:
@@
 F 0 "R301" H 4482 2904 50  0000 R CNN
 F 1 "330" H 4482 2995 50  0000 R CNN
-F 2 "" H 4550 2950 50  0001 C CNN
+F 2 "Resistor_SMD:R_0402_1005Metric" H 4550 2950 50  0001 C CNN
 F 3 "~" H 4550 2950 50  0001 C CNN
 	1    4550 2950
@@
 F 0 "R302" H 4482 3254 50  0000 R CNN
 F 1 "2k7" H 4482 3345 50  0000 R CNN
-F 2 "" H 4550 3300 50  0001 C CNN
+F 2 "Resistor_SMD:R_0603_1608Metric" H 4550 3300 50  0001 C CNN
 F 3 "~" H 4550 3300 50  0001 C CNN
 	1    4550 3300
@@
 Wire Wire Line
 	4550 3500 4550 3400
-Text HLabel 5200 3100 2    50   Output ~ 0
+Text HLabel 5400 3400 2    50   Output ~ 0
 PROXY_SENS
+$Comp
+L Device:R_Small_US R303
+U 1 1 5EF2D9C7
+P 5250 3200
+F 0 "R303" H 5318 3246 50  0000 L CNN
+F 1 "30k" H 5318 3155 50  0000 L CNN
+F 2 "Resistor_SMD:R_0603_1608Metric" H 5250 3200 50  0001 C CNN
+F 3 "~" H 5250 3200 50  0001 C CNN
+	1    5250 3200
+	1    0    0    -1
+$EndComp
+$Comp
+L Device:R_Small_US R304
+U 1 1 5EF2E0D4
+P 5250 3600
+F 0 "R304" H 5318 3646 50  0000 L CNN
+F 1 "82k" H 5318 3555 50  0000 L CNN
+F 2 "Resistor_SMD:R_0603_1608Metric" H 5250 3600 50  0001 C CNN
+F 3 "~" H 5250 3600 50  0001 C CNN
+	1    5250 3600
+	1    0    0    -1
+$EndComp
 Wire Wire Line
-	4550 3100 5200 3100
+	4550 3100 5250 3100
+Wire Wire Line
+	5250 3500 5250 3400
+Wire Wire Line
+	5400 3400 5250 3400
+Connection ~ 5250 3400
+Wire Wire Line
+	5250 3400 5250 3300
+$Comp
+L power:GND #PWR0303
+U 1 1 5EF2E6D1
+P 5250 3700
+F 0 "#PWR0303" H 5250 3450 50  0001 C CNN
+F 1 "GND" H 5255 3527 50  0000 C CNN
+F 2 "" H 5250 3700 50  0001 C CNN
+F 3 "" H 5250 3700 50  0001 C CNN
+	1    5250 3700
+	1    0    0    -1
+$EndComp
 $EndSCHEMATC
