File: PHY_fixed.sch (KiCad schematic (older format))
At the start: 45 parts, among them J801 RJMG1BD3B8K1ANR, U801 AMS1117-3.3, U802 DP83848C

Commit message: Add files via upload
Parts:
- R1016: footprint Resistor_SMD:R_0402_1005Metric -> Resistor_SMD:R_0603_1608Metric
Changed lines of the file:
@@
 F 0 "R1016" V 8350 3550 50  0000 L CNN
 F 1 "180" V 8350 3400 50  0000 L CNN
-F 2 "Resistor_SMD:R_0402_1005Metric" H 8250 3500 50  0001 C CNN
+F 2 "Resistor_SMD:R_0603_1608Metric" H 8250 3500 50  0001 C CNN
 F 3 "~" H 8250 3500 50  0001 C CNN
 	1    8250 3500
