File: polit_evse.sch (KiCad schematic (older format))
At the start: 22 parts, among them Q801 AO3400A, Q802 AO3401A, U801 LM358, U802 MEA1D0515SC

Commit message: Add files via upload
Parts:
- C801, C802: footprint (none) -> Capacitor_SMD:C_0402_1005Metric
- D801: footprint (none) -> Diode_SMD:D_SOD-123
- D802, D803: footprint (none) -> LED_SMD:LED_0805_2012Metric
- Q801: footprint (none) -> Package_TO_SOT_SMD:SOT-23
- R801, R802, R803, R804, R809, R810, R811, R812, R813: footprint (none) -> Resistor_SMD:R_0402_1005Metric
- R805, R806, R807, R808: footprint (none) -> Resistor_SMD:R_0603_1608Metric
- U801: footprint (none) -> Package_SO:SOIC-8_3.9x4.9mm_P1.27mm
- U802: footprint (none) -> MEA1D0515SC:MEA1D0515SC
Changed lines of the file:
@@
 F 0 "U802" H 5775 5015 50  0000 C CNN
 F 1 "MEA1D0515SC" H 5775 4924 50  0000 C CNN
-F 2 "" H 5650 4550 50  0001 C CNN
+F 2 "MEA1D0515SC:MEA1D0515SC" H 5650 4550 50  0001 C CNN
 F 3 "" H 5650 4550 50  0001 C CNN
 	1    5650 4550
@@
 F 0 "U801" H 5650 2617 50  0000 C CNN
 F 1 "LM358" H 5650 2526 50  0000 C CNN
-F 2 "" H 5650 2250 50  0001 C CNN
+F 2 "Package_SO:SOIC-8_3.9x4.9mm_P1.27mm" H 5650 2250 50  0001 C CNN
 F 3 "http://www.ti.com/lit/ds/symlink/lm2904-n.pdf" H 5650 2250 50  0001 C CNN
 	1    5650 2250
@@
 F 0 "U801" H 7658 4446 50  0000 L CNN
 F 1 "LM358" H 7658 4355 50  0000 L CNN
-F 2 "" H 7700 4400 50  0001 C CNN
+F 2 "Package_SO:SOIC-8_3.9x4.9mm_P1.27mm" H 7700 4400 50  0001 C CNN
 F 3 "http://www.ti.com/lit/ds/symlink/lm2904-n.pdf" H 7700 4400 50  0001 C CNN
 	3    7700 4400
@@
 F 0 "R812" H 7068 4096 50  0000 L CNN
 F 1 "2k2" H 7068 4005 50  0000 L CNN
-F 2 "" H 7000 4050 50  0001 C CNN
+F 2 "Resistor_SMD:R_0402_1005Metric" H 7000 4050 50  0001 C CNN
 F 3 "~" H 7000 4050 50  0001 C CNN
 	1    7000 4050
@@
 F 0 "R813" H 7068 4746 50  0000 L CNN
 F 1 "2k2" H 7068 4655 50  0000 L CNN
-F 2 "" H 7000 4700 50  0001 C CNN
+F 2 "Resistor_SMD:R_0402_1005Metric" H 7000 4700 50  0001 C CNN
 F 3 "~" H 7000 4700 50  0001 C CNN
 	1    7000 4700
@@
 F 0 "D802" V 7046 4180 50  0000 R CNN
 F 1 "LED_0805" V 6955 4180 50  0000 R CNN
-F 2 "" V 7000 4250 50  0001 C CNN
+F 2 "LED_SMD:LED_0805_2012Metric" V 7000 4250 50  0001 C CNN
 F 3 "~" V 7000 4250 50  0001 C CNN
 	1    7000 4250
@@
 F 0 "D803" V 7046 4830 50  0000 R CNN
 F 1 "LED_0805" V 6955 4830 50  0000 R CNN
-F 2 "" V 7000 4900 50  0001 C CNN
+F 2 "LED_SMD:LED_0805_2012Metric" V 7000 4900 50  0001 C CNN
 F 3 "~" V 7000 4900 50  0001 C CNN
 	1    7000 4900
@@
 F 0 "C801" H 6792 4196 50  0000 L CNN
 F 1 "1u" H 6792 4105 50  0000 L CNN
-F 2 "" H 6700 4150 50  0001 C CNN
+F 2 "Capacitor_SMD:C_0402_1005Metric" H 6700 4150 50  0001 C CNN
 F 3 "~" H 6700 4150 50  0001 C CNN
 	1    6700 4150
@@
 F 0 "C802" H 6792 4846 50  0000 L CNN
 F 1 "1u" H 6792 4755 50  0000 L CNN
-F 2 "" H 6700 4800 50  0001 C CNN
+F 2 "Capacitor_SMD:C_0402_1005Metric" H 6700 4800 50  0001 C CNN
 F 3 "~" H 6700 4800 50  0001 C CNN
 	1    6700 4800
@@
 F 0 "R809" V 6755 2250 50  0000 C CNN
 F 1 "1k" V 6664 2250 50  0000 C CNN
-F 2 "" H 6550 2250 50  0001 C CNN
+F 2 "Resistor_SMD:R_0402_1005Metric" H 6550 2250 50  0001 C CNN
 F 3 "~" H 6550 2250 50  0001 C CNN
 	1    6550 2250
@@
 F 0 "R806" V 5305 2550 50  0000 C CNN
 F 1 "11k" V 5214 2550 50  0000 C CNN
-F 2 "" H 5100 2550 50  0001 C CNN
+F 2 "Resistor_SMD:R_0603_1608Metric" H 5100 2550 50  0001 C CNN
 F 3 "~" H 5100 2550 50  0001 C CNN
 	1    5100 2550
@@
 F 0 "R807" H 5368 2796 50  0000 L CNN
 F 1 "82k" H 5368 2705 50  0000 L CNN
-F 2 "" H 5300 2750 50  0001 C CNN
+F 2 "Resistor_SMD:R_0603_1608Metric" H 5300 2750 50  0001 C CNN
 F 3 "~" H 5300 2750 50  0001 C CNN
 	1    5300 2750
@@
 F 0 "R805" V 5305 2150 50  0000 C CNN
 F 1 "11k" V 5214 2150 50  0000 C CNN
-F 2 "" H 5100 2150 50  0001 C CNN
+F 2 "Resistor_SMD:R_0603_1608Metric" H 5100 2150 50  0001 C CNN
 F 3 "~" H 5100 2150 50  0001 C CNN
 	1    5100 2150
@@
 F 0 "R808" V 5855 1800 50  0000 C CNN
 F 1 "82k" V 5764 1800 50  0000 C CNN
-F 2 "" H 5650 1800 50  0001 C CNN
+F 2 "Resistor_SMD:R_0603_1608Metric" H 5650 1800 50  0001 C CNN
 F 3 "~" H 5650 1800 50  0001 C CNN
 	1    5650 1800
@@
 F 0 "R804" H 4818 2796 50  0000 L CNN
 F 1 "330" H 4818 2705 50  0000 L CNN
-F 2 "" H 4750 2750 50  0001 C CNN
+F 2 "Resistor_SMD:R_0402_1005Metric" H 4750 2750 50  0001 C CNN
 F 3 "~" H 4750 2750 50  0001 C CNN
 	1    4750 2750
@@
 F 0 "R803" V 4395 2550 50  0000 C CNN
 F 1 "680" V 4486 2550 50  0000 C CNN
-F 2 "" H 4600 2550 50  0001 C CNN
+F 2 "Resistor_SMD:R_0402_1005Metric" H 4600 2550 50  0001 C CNN
 F 3 "~" H 4600 2550 50  0001 C CNN
 	1    4600 2550
@@
 F 0 "R811" H 6782 3054 50  0000 R CNN
 F 1 "18k" H 6782 3145 50  0000 R CNN
-F 2 "" H 6850 3100 50  0001 C CNN
+F 2 "Resistor_SMD:R_0402_1005Metric" H 6850 3100 50  0001 C CNN
 F 3 "~" H 6850 3100 50  0001 C CNN
 	1    6850 3100
@@
 F 0 "R810" H 6782 2704 50  0000 R CNN
 F 1 "47k" H 6782 2795 50  0000 R CNN
-F 2 "" H 6850 2750 50  0001 C CNN
+F 2 "Resistor_SMD:R_0402_1005Metric" H 6850 2750 50  0001 C CNN
 F 3 "~" H 6850 2750 50  0001 C CNN
 	1    6850 2750
@@
 F 0 "D801" V 6896 2380 50  0000 R CNN
 F 1 "B5819W" V 6805 2380 50  0000 R CNN
-F 2 "" V 6850 2450 50  0001 C CNN
+F 2 "Diode_SMD:D_SOD-123" V 6850 2450 50  0001 C CNN
 F 3 "~" V 6850 2450 50  0001 C CNN
 	1    6850 2450
@@
 F 0 "Q801" H 4705 5146 50  0000 L CNN
 F 1 "AO3400A" H 4705 5055 50  0000 L CNN
-F 2 "" H 4700 5200 50  0001 C CNN
+F 2 "Package_TO_SOT_SMD:SOT-23" H 4700 5200 50  0001 C CNN
 F 3 "~" H 4500 5100 50  0001 C CNN
 	1    4500 5100
@@
 F 0 "R801" H 4318 4596 50  0000 L CNN
 F 1 "10k" H 4318 4505 50  0000 L CNN
-F 2 "" H 4250 4550 50  0001 C CNN
+F 2 "Resistor_SMD:R_0402_1005Metric" H 4250 4550 50  0001 C CNN
 F 3 "~" H 4250 4550 50  0001 C CNN
 	1    4250 4550
@@
 F 0 "R802" H 4318 5346 50  0000 L CNN
 F 1 "10k" H 4318 5255 50  0000 L CNN
-F 2 "" H 4250 5300 50  0001 C CNN
+F 2 "Resistor_SMD:R_0402_1005Metric" H 4250 5300 50  0001 C CNN
 F 3 "~" H 4250 5300 50  0001 C CNN
 	1    4250 5300

Commit message: Submited for production & smt assembly
v0.01
Parts:
- C801, C802: footprint Capacitor_SMD:C_0402_1005Metric -> Capacitor_SMD:C_0805_2012Metric
Changed lines of the file:
@@
 $Descr A4 11693 8268
 encoding utf-8
-Sheet 8 10
+Sheet 7 10
 Title ""
 Date ""
@@
 F 0 "C801" H 6792 4196 50  0000 L CNN
 F 1 "1u" H 6792 4105 50  0000 L CNN
-F 2 "Capacitor_SMD:C_0402_1005Metric" H 6700 4150 50  0001 C CNN
+F 2 "Capacitor_SMD:C_0805_2012Metric" H 6700 4150 50  0001 C CNN
 F 3 "~" H 6700 4150 50  0001 C CNN
 	1    6700 4150
@@
 F 0 "C802" H 6792 4846 50  0000 L CNN
 F 1 "1u" H 6792 4755 50  0000 L CNN
-F 2 "Capacitor_SMD:C_0402_1005Metric" H 6700 4800 50  0001 C CNN
+F 2 "Capacitor_SMD:C_0805_2012Metric" H 6700 4800 50  0001 C CNN
 F 3 "~" H 6700 4800 50  0001 C CNN
 	1    6700 4800
