File: stm32.sch (KiCad schematic (older format))
At the start: 55 parts, among them J701 BOOT1, J702 BOOT0, J703 SWD, SW701 TS-1187A-C-E-B, SW702 TS-1187A-C-E-B, SW703 TS-1187A-C-E-B, SW704 TS-1187A-C-E-B, SW705 TS-1187A-C-E-B, U701 AMS1117-3.3, U702 STM32F429ZITx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

Commit message: Add files via upload
Parts:
- C701, C702, C703, C704, C705, C706, C707, C708, C709, C710, C711, C712, C713, C714, C715, C716, C717, C718, C719, C720, C721, C722, C723: footprint (none) -> Capacitor_SMD:C_0402_1005Metric
- D701, D702, D703, D704, D705: footprint (none) -> LED_SMD:LED_0805_2012Metric
- FB701: footprint (none) -> Inductor_SMD:L_0805_2012Metric
- J701, J702: footprint (none) -> Connector_PinHeader_2.54mm:PinHeader_1x03_P2.54mm_Vertical
- J703: footprint (none) -> Connector_PinHeader_2.54mm:PinHeader_2x05_P2.54mm_Vertical
- R701, R702, R703, R704, R705, R706, R707, R708, R709, R710, R711, R712, R713, R714, R715: footprint (none) -> Resistor_SMD:R_0402_1005Metric
- SW701, SW702, SW703, SW704, SW705: footprint (none) -> TS-1187A-C-E-B:TS-1187A-C-E-B
- Y701: footprint (none) -> Crystal:Crystal_SMD_3225-4Pin_3.2x2.5mm

Commit message: Submited for production & smt assembly
v0.01
Parts:
- C706, C712, C714: footprint Capacitor_SMD:C_0402_1005Metric -> Capacitor_SMD:C_0603_1608Metric
- R707: footprint Resistor_SMD:R_0402_1005Metric -> Resistor_SMD:R_0805_2012Metric
Connections:
- net EVSE_PUBU is gone; now on net EV_ENABLE_PLC: U702.86 (PD15)
- net BTN0: no longer SW702.3
- net BTN1: no longer SW703.3
- net BTN2: no longer SW704.3
- net BTN3: no longer SW705.3
- net EVSE_ENABLE_PLC: now also U702.92 (PG7); no longer U702.8 (PC14)
- net EVSE_PILOT_EN: now also U702.93 (PG8); no longer U702.80 (PD11)
- net EVSE_PILOT_PWM: now also U702.91 (PG6); no longer U702.82 (PD13)
- net EVSE_PLC_RESET_N: now also U702.68 (PE15); no longer U702.76 (PB15)
- net EV_ENABLE_PLC: no longer U702.9 (PC15)
- net NRST: no longer SW701.1
- net PHY_PDOWN: now also U702.55 (PF15); no longer U702.101 (PA9)
- net SPI1_CS: now also U702.76 (PB15); no longer U702.40 (PA4)
- net SPI2_CS: now also U702.66 (PE13); no longer U702.140 (PB9)
- net SPI2_INT: now also U702.67 (PE14); no longer U702.78 (PD9)
- net STM_3V3: no longer SW702.4, SW703.4, SW704.4, SW705.4
- net ~PHY_RESET: now also U702.50 (PF12); no longer U702.100 (PA8)
- net EVSE_CONNECT_T1: now reaches U702.88 (PG3)
- net EVSE_CONNECT_T2: now reaches U702.89 (PG4)
- net EVSE_PUBU_T1: now reaches U702.90 (PG5)
- net EVSE_PROXY: no longer names the net of U702.85 (PD14)
- no-connect marks 64 -> 72
Other:
- moved on the sheet: C703, C704, FB701, R708, R709, R710, R711, SW702, SW703, SW704, SW705
